File: BatteryCharger/BatteryCharger.sch (KiCad schematic (older format))
At the start: 29 parts

Commit message: Created sch
Parts:
- removed U?: BQ24650, symbol BQ24650:BQ24650
- added Rsr: R, symbol Device:R
- added U: BQ24650, symbol BQ24650:BQ24650
- D1: renamed from D?; value D -> D1
- D2: renamed from D?; value D_Schottky -> D2
- D?: value LED -> D4
- D?: value LED -> D3
- gave numbers to parts that had none: 22
Connections:
- net at D2.1 (K): now also C?.1, U.16 (BTST)
- net at D2.2 (A): now also C4.2, U.12 (REGN)
- net at D1.1 (K): now also C6.1, Q1.1 (D), R6.2
- net VS: now reaches D1.2 (A)
- net VS: now also R3.1, R5.1, R7.2, R8.2
- net at D?.1 (K): now also U.5 (STAT2)
- net at D?.2 (A): now also R8.1
- net at D?.1 (K): now also U.3 (STAT1)
- net at D?.2 (A): now also R7.1
- net GND: now reaches C1.1
- net GND: now also C2.2, C3.2, C4.1, C6.2, C8.2, C9.2, Q2.3 (S), Q2.4 (B), Q3.3 (S), Q3.4 (B), R1.2, R10.2, R?.2, U.11 (GND)
- net at C1.2: now also R5.2
- net at C3.1: now also R9.1, U.6 (VREF), U.7 (TERM_EN)
- net BatteryPack: now reaches C10.1
- net BatteryPack: now also C7.2, C8.1, C9.1, R2.1, Rsr.1, U.9 (SRN)
- net at C10.2: now also R1.1, R2.2, U.8 (VFB)
- net at C7.1: now also L1.2, Rsr.2, U.10 (SRP)
- net at C?.2: now also L1.1, Q1.3 (S), Q1.4 (B), Q2.1 (D), U.14 (PH)
- net at C2.1: now also R6.1, U.1 (VCC)
- net PackThermistor: now reaches R9.2
- net PackThermistor: now also R10.1, U.4 (TS)
- net at R?.1: now also Q3.1 (D), R3.2, U.2 (MPPSET)
- net at Q2.2 (G): now also U.13 (LODRV)
- net at Q1.2 (G): now also U.15 (HIDRV)
Other:
- note added: "(In typical application) Solar Cell Half Panel"
- note added: "BQ24650 Typical Application Schematic"
- moved on the sheet: C1, C10, C2, C3, C4, C6, C7, C8, C9, C?, L1, Q1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

Commit message: Populated most componentse
Parts:
- removed C3: C_Small, symbol Device:C_Small
- removed D1: D1, symbol Device:D
- removed Q1, Q2, Q3: MNMOS, symbol pspice:MNMOS
- removed R3, R?: R, symbol Device:R
- added D1, D5: 10V, symbol Device:D_Zener
- added Q1, Q2: 40V 10A 10mO, symbol Device:Q_NMOS_DGS
- added Q3: Q_NMOS_DGS, symbol Device:Q_NMOS_DGS
- added Q4, Q5: 40V 10A 10mO, symbol Device:Q_PMOS_DGS
- added Q6: 2N2222A, symbol Device:Q_NPN_BEC
- added R10, R13, R14: 10k, symbol Device:R
- added R9: 100k, symbol Device:R
- C1: value C_Small -> 2.2u
- C10: value C_Small -> 22p
- C2, C4: value C_Small -> 1u
- C5: renamed from C?; value C_Small -> 0.1u
- C6, C8: value C_Small -> 10u
- C7: value C_Small -> 0.1u
- C9: value C_Small -> 4.7u
- D?: value D4 -> D4 (grn)
- D?: value D3 -> D3 (yel)
- L1: value L -> 10u
- R1: value R -> 160k
- R2: value R -> 910k
- R5: value R -> 2
- R6: value R -> 10
- R7, R8: value R -> 10k
- Rsr: value R -> 20m
- renumbered R9 to R11, R10 to R12
Connections:
- net GND: now also D5.2 (A), Q2.3 (S), Q3.3 (S), Q6.3 (C), R9.2
- net VS: now also Q4.1 (D)
- net at C6.1: now also R6.1, D1.1 (K), Q1.1 (D), Q4.3 (S); no longer R6.2
- net at R11.1, U.6 (VREF), U.7 (TERM_EN): now also R10.1
- net at C5.2, L1.1, U.14 (PH): now also Q1.3 (S), Q2.1 (D)
- net at C2.1, U.1 (VCC): now also R6.2; no longer R6.1
- net at U.2 (MPPSET): now also Q3.1 (D), R10.2
- net at U.13 (LODRV): now also Q2.2 (G)
- net at U.15 (HIDRV): now also Q1.2 (G)
- net BatteryPack: no longer names the net of C10.1, C7.2, C8.1, C9.1, R2.1, Rsr.1, U.9 (SRN)
- net BatteryPack: now also Q5.3 (S), R13.1
- new net: D1.2 (A), Q4.2 (G), R9.1
- new net: Q5.2 (G), Q6.2 (E), R13.2
- new net: D5.1 (K), Q6.1 (B), R14.2
- new net BatteryPosTerminal: Q5.1 (D), R14.1
- new net ~CE: Q3.2 (G)
Other:
- note removed: "(In typical application) Solar Cell Half Panel"
- moved on the sheet: C1, C10, C4, C5, C6, R5, R6
