File: BatteryCharger/BatteryCharger.sch (KiCad schematic (older format))
At the start: 35 parts, among them Q1 40V 10A 10mO, Q2 40V 10A 10mO, Q3 Q_NMOS_DGS, Q4 40V 10A 10mO, Q5 40V 10A 10mO, Q6 2N2222A

Commit message: Schematic finalizations
Added dual channel mosfet symbols; added test points; added a Vdiv array for TS pin; and added jumper resistors between HI/LODRV and their Nfets.
Parts:
- removed Q1, Q2: 40V 10A 10mO, symbol Device:Q_NMOS_DGS
- removed Q3: Q_NMOS_DGS, symbol Device:Q_NMOS_DGS
- removed Q4, Q5: 40V 10A 10mO, symbol Device:Q_PMOS_DGS
- added Q1: Si7288DP, symbol DualChannelMOSFET:Si7288DP
- added Q2: Si4949DY, symbol DualChannelMOSFET:Si4949DY
- added Q4: 2N2222A, symbol Device:Q_NPN_BEC
- added R15, R4: 0, symbol Device:R
- added R16, R3: 10k, symbol Device:R
- added TP1, TP2, TP3, TP4, TP5, TP6, TP7, TP8, TP9: TestPoint, symbol Connector:TestPoint
- R11, R12: value R -> 10k
- U1: renamed from U; symbol BQ24650:BQ24650 -> BatteryCharger-rescue:BQ24650-BQ24650
- gave numbers to parts that had none: 2
- renumbered Q6 to Q3, Rsr to Rsr1
Connections:
- net labels removed: PackThermistor
- wire segments 111 -> 131
Other:
- moved on the sheet: C1, C10, C2, C4, C5, C6, C7, C8, C9, D1, D5, L1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

Commit message: Pre-transition to git
Parts:
- removed Q1: Si7288DP, symbol DualChannelMOSFET:Si7288DP
- removed Q2: Si4949DY, symbol DualChannelMOSFET:Si4949DY
- added D6: 10V, symbol Device:D_Zener
- added Q2, Q5: Q_PMOS_GDS, symbol Device:Q_PMOS_GDS
- C8: value 10u -> 40u
- L1: value 10u -> 3.3u
- Rsr1: value 20m -> 5m
- renumbered TP5 to +Vbat, TP6 to HNmosG, TP7 to LNmosG, TP8 to PH, TP4 to Srn, TP9 to Srp, TP3 to SwHigh, TP2 to Vfb, TP1 to Vref
Connections:
- net labels removed: ~CE
Other:
- note added: "BQ24650 Charger Sch"
- note removed: "BQ24650 Typical Application Schematic"
- moved on the sheet: D5, Q3, Q4, R13, R3

Commit message: Prettified schematic and updated MOS/NPN symbols.  Added expansion for multiple output capacitors.
Parts:
- removed C8: 40u, symbol Device:C_Small
- added C11, C12, C3, C8: 10u, symbol Device:CP_Small
- added D7: Red, symbol Device:LED
- added D8: Green, symbol Device:LED
- added Q1, Q6: Q_NMOS_GDS, symbol Device:Q_NMOS_GDS
- added R17, R18: 10k, symbol Device:R
- added SW1: SW_DPDT_x2, symbol Switch:SW_DPDT_x2
- added Srn1: TestPoint, symbol Connector:TestPoint
- D3: value D3 (yel) -> Yellow
- D4: value D4 (grn) -> Green
- U1: symbol BatteryCharger-rescue:BQ24650-BQ24650 -> BQ24650:BQ24650
- renumbered +Vbat to +Vbat1, HNmosG to HNmos, LNmosG to LNmos, PH to PH1, Srn to Srn2, Srp to Srp1, SwHigh to SwHigh1, Vfb to Vfb1, Vref to Vref1
Connections:
- wire segments 131 -> 159
Other:
- note added: "Charge Disable:\nTurn Switch to show red to disable charge"
- moved on the sheet: +Vbat1, C1, C10, C2, C4, C5, C6, C7, C9, D1, D5, D6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
